Commit message: modify arm simulations and update chassis sim

File: Software_control/Worksapce_folder/Robot_arm_ws/src/mycobot280_pi/urdf/mycobot_280_gazebo.urdf (robot description, URDF)
Before this commit: robot mycobot280_pi, 9 links, 8 joints
Links:
- link g_base: geometry collision box size=0.08 0.08 0.04; visual mesh filename=package://mycobot280_pi/urdf/meshes/G_base.dae
- link joint1: geometry collision box size=0.06 0.06 0.06; visual mesh filename=package://mycobot280_pi/urdf/meshes/joint1.stl
- link joint2: geometry collision box size=0.05 0.05 0.08; visual mesh filename=package://mycobot280_pi/urdf/meshes/joint2.dae
- link joint3: geometry collision box size=0.05 0.05 0.06; visual mesh filename=package://mycobot280_pi/urdf/meshes/joint3.dae
- link joint4: geometry collision box size=0.05 0.05 0.05; visual mesh filename=package://mycobot280_pi/urdf/meshes/joint4.dae
- link joint5: geometry collision box size=0.04 0.04 0.04; visual mesh filename=package://mycobot280_pi/urdf/meshes/joint5.stl
- link joint6: geometry collision box size=0.04 0.04 0.04; visual mesh filename=package://mycobot280_pi/urdf/meshes/joint6.dae
- link joint6_flange: geometry collision box size=0.03 0.03 0.03; visual mesh filename=package://mycobot280_pi/urdf/meshes/joint7.dae
