Commit message: can get  bin but not accurate

File: System_integration/Ver01_ws/src/leo_custom_simulation/urdf/leo_with_lidar_camera.urdf.xacro (robot description, xacro)
@@ -68,5 +68,5 @@
     <parent link="base_link"/>
     <child link="D435i_camera_link"/>
-    <origin xyz="0.14813 -0.027 0.05957" rpy="0.0 0.0 0.0"/>
+    <origin xyz="0.14813 -0.027 0.05957" rpy="0.0 0.34 0.0"/>
   </joint>
   <!-- depth camera frame -->
